File: eurorack/Cwejman/VCA-4MX/Cwejman_VCA-4MX_Template.kicad_pcb (KiCad board)
At the start: 2 copper layers, 2 parts

Commit message: SVG correction
corrected SVG export size.
Parts:
- removed REF**: BKM_Signature_3, Eurorack Footprints:BKM_Signature_3
- removed REF**: Fish_mark_1, Eurorack Footprints:Fish_mark_1
Routing:
- removed copper zone on F.Cu, net (none)
